Commit message: Xaxafour/gazebo plugin (#52)
* Implementation of gazebo plugin with strategy 3

* Update plugin controller structure

* Added switching x models via urdf

* Update model names and gear ratios

* Implemented multiple control strategies

* Added low pass filter

* Added setting command lifetime and changed symbol for x models to hyphen

* Fix effort control

* Clean up plugin files

* Reset feedback frequency for gazebo and change gazebo launch to use a basic example

* Remove launch files from plugin

File: hebiros_description/urdf/1_dof.xacro (robot description, xacro)
@@ -43,10 +43,6 @@
   </joint>
   <!-- joints -->
-  <xacro:x5 joint="HEBI/base" child="shoulder_bracket" model="X5_4"/>
-  <xacro:x_wrist_bracket name="shoulder_bracket" child="HEBI/shoulder"/>
-  <xacro:x5 joint="HEBI/shoulder" child="shoulder_elbow" model="X5_4"/>
-  <xacro:x_tube_link name="shoulder_elbow" child="HEBI/elbow" length="0.33" twist="0.7"/>
-  <xacro:x5 joint="HEBI/elbow" child="elbow_end" model="X5_4"/>
-  <xacro:x_tube_link name="elbow_end" child="end_effector" length="0.325" twist="0.6"/>
+  <xacro:x5 joint="HEBI/base" child="base_end" model="X5-4"/>
+  <xacro:x_tube_link name="base_end" child="end_effector" length="0.33" twist="0"/>
   <!-- end link -->
   <link name="end_effector/INPUT_INTERFACE">

File: hebiros_description/urdf/x5.xacro (robot description, xacro)
@@ -2,5 +2,6 @@
 <robot xmlns:xacro="http://www.ros.org/wiki/xacro">
   <!-- NOTE: joint must match the name of the module -->
-  <xacro:macro name="x5" params="joint child">
+  <xacro:macro name="x5" params="joint child model">
+  <xacro:property name="model_name" value="${model}"/>
     <link name="${joint}/INPUT_INTERFACE">
       <visual>
@@ -23,12 +24,34 @@
       </inertial>
     </link>
-    <joint name="${joint}" type="revolute">
-      <parent link="${joint}/INPUT_INTERFACE"/>
-      <child link="${child}/INPUT_INTERFACE"/>
-      <origin xyz="0 0 0.031" rpy="0 0 0"/>
-      <axis xyz="0 0 1"/>
-      <limit effort="9.0" lower="-10.0" upper="10.0" velocity="2.208932"/>
-      <dynamics damping="0.2" friction="0.2"/>
-    </joint>
+    <xacro:if value="${model_name == 'X5_1'}">
+      <joint name="${joint}/X5_1" type="revolute">
+        <parent link="${joint}/INPUT_INTERFACE"/>
+        <child link="${child}/INPUT_INTERFACE"/>
+        <origin xyz="0 0 0.031" rpy="0 0 0"/>
+        <axis xyz="0 0 1"/>
+        <limit effort="9.0" lower="-10.0" upper="10.0" velocity="2.208932"/>
+        <dynamics damping="0.5" friction="0.5"/>
+      </joint>
+    </xacro:if>
+    <xacro:if value="${model_name == 'X5_4'}">
+      <joint name="${joint}/X5_4" type="revolute">
+        <parent link="${joint}/INPUT_INTERFACE"/>
+        <child link="${child}/INPUT_INTERFACE"/>
+        <origin xyz="0 0 0.031" rpy="0 0 0"/>
+        <axis xyz="0 0 1"/>
+        <limit effort="9.0" lower="-10.0" upper="10.0" velocity="2.208932"/>
+        <dynamics damping="0.5" friction="0.5"/>
+      </joint>
+    </xacro:if>
+    <xacro:if value="${model_name == 'X5_9'}">
+      <joint name="${joint}/X5_9" type="revolute">
+        <parent link="${joint}/INPUT_INTERFACE"/>
+        <child link="${child}/INPUT_INTERFACE"/>
+        <origin xyz="0 0 0.031" rpy="0 0 0"/>
+        <axis xyz="0 0 1"/>
+        <limit effort="9.0" lower="-10.0" upper="10.0" velocity="2.208932"/>
+        <dynamics damping="0.5" friction="0.5"/>
+      </joint>
+    </xacro:if>
     <transmission name="${joint}/transmission">
     <type>transmission_interface/SimpleTransmission</type>

File: hebiros_description/urdf/x_demo.urdf (robot description, URDF)
Before this commit: robot arm_demo, 9 links, 8 joints
Links:
- link elbow_end/INPUT_INTERFACE: geometry collision cylinder length=0.325 radius=.015875; collision mesh filename=package://hebiros_description/meshes/x_mounting_bracket.stl
- link shoulder_elbow/INPUT_INTERFACE: geometry collision cylinder length=0.33 radius=.015875; collision mesh filename=package://hebiros_description/meshes/x_mounting_bracket.stl
Joints:
- removed joint HEBI/base
- removed joint HEBI/elbow
- removed joint HEBI/shoulder
- added joint HEBI/base/X5_4: type revolute, parent HEBI/base/INPUT_INTERFACE, child shoulder_bracket/INPUT_INTERFACE, origin xyz=0 0 0.031 rpy=0 0 0, axis 0 0 1, limit lower=-10.0 upper=10.0 effort=9.0 velocity=2.208932
- added joint HEBI/elbow/X5_4: type revolute, parent HEBI/elbow/INPUT_INTERFACE, child elbow_end/INPUT_INTERFACE, origin xyz=0 0 0.031 rpy=0 0 0, axis 0 0 1, limit lower=-10.0 upper=10.0 effort=9.0 velocity=2.208932
- added joint HEBI/shoulder/X5_4: type revolute, parent HEBI/shoulder/INPUT_INTERFACE, child shoulder_elbow/INPUT_INTERFACE, origin xyz=0 0 0.031 rpy=0 0 0, axis 0 0 1, limit lower=-10.0 upper=10.0 effort=9.0 velocity=2.208932

File: hebiros_description/urdf/x_tube_link.xacro (robot description, xacro)
@@ -14,5 +14,5 @@
         <origin xyz="${-length/2-.0254} 0 .016075" rpy="0 1.57075 0" />
         <geometry>
-          <cylinder length="${length}" radius=".015875" />
+          <cylinder length="${length-.0254}" radius=".015875" />
         </geometry>
         <xacro:silver_material/>
